File: TSOC_NEOLED/TSOC_NEOLED.brd (EAGLE design)
At the start: 53.3 x 30.5 mm, 49 parts, among them U1 SN74HC245PW, U2 CY8C42XX-44PIN

Commit message: update descriptions
Parts:
- moved C9 0.57 mm to (38.9, 22.4)
- moved R2 0.51 mm to (5.33, 4.06)
Routing:
- net VEXT: track 80.2 -> 80.8 mm
- net P3_0: track 41.7 -> 41.2 mm
- net VCC: track 121.9 -> 122.5 mm
Changed lines of the file:
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@@
 <layer number="37" name="tTest" color="7" fill="1" visible="no" active="yes"/>
 <layer number="38" name="bTest" color="7" fill="1" visible="no" active="yes"/>
-<layer number="39" name="tKeepout" color="4" fill="11" visible="no" active="yes"/>
-<layer number="40" name="bKeepout" color="1" fill="11" visible="no" active="yes"/>
-<layer number="41" name="tRestrict" color="4" fill="10" visible="no" active="yes"/>
-<layer number="42" name="bRestrict" color="1" fill="10" visible="no" active="yes"/>
-<layer number="43" name="vRestrict" color="2" fill="10" visible="no" active="yes"/>
-<layer number="44" name="Drills" color="7" fill="1" visible="no" active="yes"/>
-<layer number="45" name="Holes" color="7" fill="1" visible="no" active="yes"/>
-<layer number="46" name="Milling" color="3" fill="1" visible="no" active="yes"/>
+<layer number="39" name="tKeepout" color="4" fill="11" visible="yes" active="yes"/>
+<layer number="40" name="bKeepout" color="1" fill="11" visible="yes" active="yes"/>
+<layer number="41" name="tRestrict" color="4" fill="10" visible="yes" active="yes"/>
+<layer number="42" name="bRestrict" color="1" fill="10" visible="yes" active="yes"/>
+<layer number="43" name="vRestrict" color="2" fill="10" visible="yes" active="yes"/>
+<layer number="44" name="Drills" color="7" fill="1" visible="yes" active="yes"/>
+<layer number="45" name="Holes" color="7" fill="1" visible="yes" active="yes"/>
+<layer number="46" name="Milling" color="3" fill="1" visible="yes" active="yes"/>
 <layer number="47" name="Measures" color="7" fill="1" visible="no" active="yes"/>
 <layer number="48" name="Document" color="7" fill="1" visible="no" active="yes"/>
@@
 <board>
 <plain>
-<text x="45.72" y="26.162" size="0.8128" layer="21" font="vector" ratio="14">SIG</text>
+<text x="45.72" y="25.654" size="0.8128" layer="21" font="vector" ratio="14">SIG</text>
 <text x="48.26" y="25.654" size="0.8128" layer="21" font="vector" ratio="14">PWR</text>
 <text x="50.8" y="25.654" size="0.8128" layer="21" font="vector" ratio="14">GND</text>
@@
 <attribute name="VALUE" x="35.687" y="19.685" size="0.6096" layer="27" font="vector" ratio="15" rot="R90"/>
 </element>
-<element name="C9" library="PatternAgents-Misc" package="0603-CAP" value="0.1uF" x="38.608" y="21.844" smashed="yes" rot="R180">
-<attribute name="NAME" x="38.227" y="23.114" size="0.6096" layer="25" font="vector" ratio="15" rot="R180"/>
-<attribute name="VALUE" x="40.005" y="23.241" size="0.6096" layer="27" font="vector" ratio="15" rot="R180"/>
+<element name="C9" library="PatternAgents-Misc" package="0603-CAP" value="0.1uF" x="38.862" y="22.352" smashed="yes" rot="R180">
+<attribute name="NAME" x="38.481" y="23.622" size="0.6096" layer="25" font="vector" ratio="15" rot="R180"/>
+<attribute name="VALUE" x="40.259" y="23.749" size="0.6096" layer="27" font="vector" ratio="15" rot="R180"/>
 </element>
 <element name="J2" library="PatternAgents-ProtoPads" package="1X08_ROUND" value="" x="46.736" y="24.13" smashed="yes" rot="R270">
@@
 <attribute name="VALUE" x="10.668" y="17.907" size="1.27" layer="27"/>
 </element>
-<element name="R2" library="PatternAgents-Misc" package="0603-RES" value="2K2" x="5.334" y="3.556" smashed="yes">
-<attribute name="NAME" x="2.159" y="3.302" size="0.6096" layer="25" font="vector" ratio="15"/>
-<attribute name="VALUE" x="3.937" y="2.159" size="0.6096" layer="27" font="vector" ratio="15"/>
+<element name="R2" library="PatternAgents-Misc" package="0603-RES" value="2K2" x="5.334" y="4.064" smashed="yes">
+<attribute name="NAME" x="2.159" y="3.81" size="0.6096" layer="25" font="vector" ratio="15"/>
+<attribute name="VALUE" x="3.937" y="2.667" size="0.6096" layer="27" font="vector" ratio="15"/>
 </element>
 <element name="R1" library="PatternAgents-Misc" package="0603-RES" value="2K2" x="5.334" y="1.778" smashed="yes">
@@
 <contactref element="C10" pad="1"/>
 <wire x1="36.322" y1="21.932" x2="37.67" y2="21.932" width="0.6096" layer="1"/>
-<wire x1="37.67" y1="21.932" x2="37.758" y2="21.844" width="0.6096" layer="1"/>
+<wire x1="37.67" y1="21.932" x2="38.012" y2="22.352" width="0.6096" layer="1"/>
 <wire x1="41.402" y1="29.464" x2="41.91" y2="29.972" width="0.6096" layer="16"/>
 <wire x1="41.91" y1="29.972" x2="43.434" y2="29.972" width="0.4064" layer="16"/>
@@
 <wire x1="10.668" y1="2.286" x2="10.668" y2="10.668" width="0.254" layer="16"/>
 <wire x1="10.668" y1="10.668" x2="10.414" y2="10.922" width="0.254" layer="16"/>
-<wire x1="6.184" y1="3.556" x2="6.184" y2="1.778" width="0.254" layer="1"/>
+<wire x1="6.184" y1="4.064" x2="6.184" y2="1.778" width="0.254" layer="1"/>
 <contactref element="R12" pad="2"/>
 <contactref element="R9" pad="2"/>
@@
 <wire x1="3.048" y1="5.334" x2="3.048" y2="19.812" width="0.254" layer="1"/>
 <contactref element="R2" pad="1"/>
-<wire x1="4.484" y1="3.556" x2="4.484" y2="4.914" width="0.254" layer="1"/>
+<wire x1="4.484" y1="4.064" x2="4.484" y2="4.914" width="0.254" layer="1"/>
 <wire x1="4.484" y1="4.914" x2="4.318" y2="5.08" width="0.254" layer="1"/>
 </signal>
@@
 <wire x1="49.022" y1="26.162" x2="49.276" y2="25.908" width="0.6096" layer="1"/>
 <wire x1="39.624" y1="25.908" x2="39.624" y2="22.01" width="0.6096" layer="1"/>
-<wire x1="39.624" y1="22.01" x2="39.458" y2="21.844" width="0.6096" layer="1"/>
+<wire x1="39.624" y1="22.01" x2="39.712" y2="22.352" width="0.6096" layer="1"/>
 <wire x1="38.989" y1="17.399" x2="38.989" y2="21.375" width="0.3048" layer="1"/>
-<wire x1="38.989" y1="21.375" x2="39.458" y2="21.844" width="0.3048" layer="1"/>
+<wire x1="38.989" y1="21.375" x2="39.712" y2="22.352" width="0.3048" layer="1"/>
 <wire x1="49.022" y1="26.162" x2="44.958" y2="26.162" width="0.6096" layer="1"/>
 <wire x1="44.958" y1="26.162" x2="39.878" y2="26.162" width="0.6096" layer="1"/>
